File: Super Starbie.kicad_sch (KiCad schematic)
At the start: 15 parts, among them J1 Conn_01x04_Pin, J2 Conn_01x08_Pin, M1 Motor_DC, Q1 Q_NMOS_DGS, U3 DHT11

Commit message: Add files via upload
Connections:
- net at U1.10 (GPIO26): now also Power_ON/OFF1.1; no longer Switch_2.1
- net at U1.12 (GPIO33): now also Switch_3.1; no longer Power_ON/OFF1.1
- net at J1.1 (Pin_1), J2.1 (Pin_1), U1.19 (3.3v)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: now also M1.1 (+)
- net at D1.1 (K), J1.2 (Pin_2), J2.2 (Pin_2)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: no longer M1.1 (+)
- net at U1.9 (GPIO27): now also Switch_2.1; no longer Switch_3.1
Other:
- moved on the sheet: D1, Power_ON/OFF1, R2, Switch_2, Switch_3
