File: PCB/Super Starbie.kicad_pcb (KiCad board)
At the start: 2 copper layers, 110 x 105 mm, 14 parts, among them J3 OLED_SH1107, J4 MPU6050, M2 Motor_DC, Q2 Q_NMOS_DGS, SW1 SW_Push, SW2 SW_Push, SW3 SW_Push, SW4 SW_Push, SW5 SW_Push, U2 esp32_Wroom_32S_30_Pins, U4 DHT11

Commit message: Add files via upload
Parts:
- moved R1 108.6 mm to (188.0, 95.0)
- moved R4 97.2 mm to (178.0, 92.5)
- moved D1 76.7 mm to (173.5, 92.0), turned to 180 degrees
- moved Q2 22.1 mm to (167.0, 88.0)
- moved U4 20.9 mm to (178.4, 87.5)
- moved J4 10.0 mm to (185.1, 96.0)
- moved M2 2.28 mm to (163.0, 29.5), turned to -90 degrees
- moved SW1 0.92 mm to (158.5, 47.6)
Connections:
- SW1 pad 1: Net-(U2-GPIO13) -> Net-(U2-GPIO14)
- SW2 pad 1: Net-(U2-GPIO14) -> Net-(U2-GPIO13)
Routing:
- net GND: track 0.00 -> 292.9 mm
- net +3.3V: track 0.00 -> 157.2 mm
- net Net-(D1-A): track 0.00 -> 72.8 mm
- net /SCL: track 0.00 -> 68.1 mm
- net Net-(U2-GPIO26): track 0.00 -> 63.5 mm
- net /SDA: track 0.00 -> 62.6 mm
- net Net-(U2-GPIO25): track 0.00 -> 56.7 mm
- net Net-(U2-GPIO4): track 0.00 -> 52.2 mm
- net Net-(U2-GPIO27): track 0.00 -> 51.7 mm
- net Net-(Q2-G): track 0.00 -> 44.5 mm
- net Net-(U2-GPIO14): track 0.00 -> 37.6 mm
- net Net-(U2-GPIO13): track 0.00 -> 29.2 mm
Other:
- outline, holes or cut-outs redrawn
